File: hardware/alpha-1/alpha.sch (KiCad schematic (older format))
At the start: 82 parts, among them J1 POWER, J2 SERIAL, P1 SWITCH_1, P2 SWITCH_2, P3 SWITCH_3, P4 SWITCH_4, P5 SWITCH_5, P6 SWITCH_6, P7 INPUTS, P8 RASPBERRY_PI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

Commit message: o Updating some footprints, laying out connectors.
Parts:
- D1, D11, D3, D5, D7: footprint Diodes_SMD:D_SMA_Handsoldering -> Diodes_SMD:D_SMA
Changed lines of the file:
@@
 F 0 "D3" H 12700 4150 50  0000 C CNN
 F 1 "S1MTR" H 12700 3950 50  0000 C CNN
-F 2 "Diodes_SMD:D_SMA_Handsoldering" H 12700 4050 50  0001 C CNN
+F 2 "Diodes_SMD:D_SMA" H 12700 4050 50  0001 C CNN
 F 3 "http://www.smc-diodes.com/propdf/S1A-S1M%20N0560%20REV.B.pdf" H 12700 4050 50  0001 C CNN
 F 4 "S1MTR" H 12700 4050 60  0001 C CNN "mpn"
@@
 F 0 "D1" H 12700 2150 50  0000 C CNN
 F 1 "S1MTR" H 12700 1950 50  0000 C CNN
-F 2 "Diodes_SMD:D_SMA_Handsoldering" H 12700 2050 50  0001 C CNN
+F 2 "Diodes_SMD:D_SMA" H 12700 2050 50  0001 C CNN
 F 3 "http://www.smc-diodes.com/propdf/S1A-S1M%20N0560%20REV.B.pdf" H 12700 2050 50  0001 C CNN
 F 4 "S1MTR" H 12700 2050 60  0001 C CNN "mpn"
@@
 F 0 "D5" H 12700 6150 50  0000 C CNN
 F 1 "S1MTR" H 12700 5950 50  0000 C CNN
-F 2 "Diodes_SMD:D_SMA_Handsoldering" H 12700 6050 50  0001 C CNN
+F 2 "Diodes_SMD:D_SMA" H 12700 6050 50  0001 C CNN
 F 3 "http://www.smc-diodes.com/propdf/S1A-S1M%20N0560%20REV.B.pdf" H 12700 6050 50  0001 C CNN
 F 4 "S1MTR" H 12700 6050 60  0001 C CNN "mpn"
@@
 F 0 "D7" H 15100 2150 50  0000 C CNN
 F 1 "S1MTR" H 15100 1950 50  0000 C CNN
-F 2 "Diodes_SMD:D_SMA_Handsoldering" H 15100 2050 50  0001 C CNN
+F 2 "Diodes_SMD:D_SMA" H 15100 2050 50  0001 C CNN
 F 3 "http://www.smc-diodes.com/propdf/S1A-S1M%20N0560%20REV.B.pdf" H 15100 2050 50  0001 C CNN
 F 4 "S1MTR" H 15100 2050 60  0001 C CNN "mpn"
@@
 F 0 "D11" H 15100 6150 50  0000 C CNN
 F 1 "S1MTR" H 15100 5950 50  0000 C CNN
-F 2 "Diodes_SMD:D_SMA_Handsoldering" H 15100 6050 50  0001 C CNN
+F 2 "Diodes_SMD:D_SMA" H 15100 6050 50  0001 C CNN
 F 3 "http://www.smc-diodes.com/propdf/S1A-S1M%20N0560%20REV.B.pdf" H 15100 6050 50  0001 C CNN
 F 4 "S1MTR" H 15100 6050 60  0001 C CNN "mpn"

Commit message: o Adjusting more footprints.
Parts:
- D9: footprint Diodes_SMD:D_SMA_Handsoldering -> Diodes_SMD:D_SMA
Changed lines of the file:
@@
 F 0 "D9" H 15100 4150 50  0000 C CNN
 F 1 "S1MTR" H 15100 3950 50  0000 C CNN
-F 2 "Diodes_SMD:D_SMA_Handsoldering" H 15100 4050 50  0001 C CNN
+F 2 "Diodes_SMD:D_SMA" H 15100 4050 50  0001 C CNN
 F 3 "http://www.smc-diodes.com/propdf/S1A-S1M%20N0560%20REV.B.pdf" H 15100 4050 50  0001 C CNN
 F 4 "S1MTR" H 15100 4050 60  0001 C CNN "mpn"
