File: hardware/alpha-2/alpha.kicad_pcb (KiCad board)
At the start: 2 copper layers, 65 x 56 mm, 95 parts, among them J1 POWER, J2 SERIAL, P1 OUTPUTS, P2 INPUTS, P3 RASPBERRY_PI, P4 12V, Q1 DMN2041L-7, Q2 DMN2041L-7, Q3 DMN2041L-7, Q4 DMN2041L-7, Q5 DMN2041L-7, Q6 DMN2041L-7, Q7 DMN2041L-7, U1 TPS54202, U2 TMP102, U3 ESP-12E

Commit message: wip, alpha-2.
Parts:
- removed R24, R25, R26: 10k, IPC7351-Nominal:RESC1005X38
- removed U2: TMP102, Bitraf:SOT-563
- added C7: 4.7u, IPC-7351-CAPC:CAPC_2012x125, F.Cu at (167.0, 113.0)
- added C8: 4.7u, IPC-7351-CAPC:CAPC_2012x125, F.Cu at (167.0, 109.0)
- added R37: 10k, IPC-7351-RESC:RESC_1005x040, F.Cu at (296.1, 102.0)
- added TP1: TEST_1P, Connectors_TestPoints:Test_Point_Pad_d1.0mm, F.Cu at (232.5, 160.1)
- added TP2: TEST_1P, Connectors_TestPoints:Test_Point_Pad_d1.0mm, F.Cu at (229.4, 160.1)
- added TP3: TEST_1P, Connectors_TestPoints:Test_Point_Pad_d1.0mm, F.Cu at (226.3, 160.1)
- added TP4: TEST_1P, Connectors_TestPoints:Test_Point_Pad_d1.0mm, F.Cu at (223.2, 160.1)
- added TP5: TEST_1P, Connectors_TestPoints:Test_Point_Pad_d1.0mm, F.Cu at (220.1, 160.1)
- added TP6: TEST_1P, Connectors_TestPoints:Test_Point_Pad_d1.0mm, F.Cu at (217.0, 160.1)
- added TP7: TEST_1P, Connectors_TestPoints:Test_Point_Pad_d1.0mm, F.Cu at (213.9, 160.1)
- added TP8: TEST_1P, Connectors_TestPoints:Test_Point_Pad_d1.0mm, F.Cu at (210.8, 160.1)
- added TP9: Vin, Connectors_TestPoints:Test_Point_Pad_d1.0mm, F.Cu at (207.8, 160.1)
- added U4: AP2114H-3.3TRG1, smd-semi:SOT-223, F.Cu at (172.4, 111.0)
- C1, C2, C3, C5, C6: footprint IPC7351-Nominal:CAPC2012X70 -> IPC-7351-CAPC:CAPC_2012x125
- C4: footprint IPC7351-Nominal:CAPC1005X55 -> IPC-7351-CAPC:CAPC_1005x050
- D10, D12, D2, D21, D22, D23, D24, D25, D26, D27, D28, D29, D30, D31, D4, D6, D8: footprint IPC7351-Nominal:LEDC3216X110 -> IPC-7351-LEDSC:LEDSC_1608x065
- J2: footprint Pin_Headers:Pin_Header_Straight_1x05_Pitch2.54mm -> Pin_Headers:Pin_Header_Straight_1x07_Pitch2.54mm
- R1, R10, R11, R12, R13, R14, R15, R16, R17, R18, R19, R2, R20, R21, R22, R23, R27, R28, R29, R3, R30, R31, R32, R33, R34, R35, R36, R4, R5, R6, R7, R8, R9: footprint IPC7351-Nominal:RESC1005X38 -> IPC-7351-RESC:RESC_1005x040
- moved R29 41.5 mm to (227.0, 125.8)
- moved R30 38.0 mm to (223.5, 125.8)
- moved R31 34.5 mm to (220.0, 125.8)
- moved R32 31.0 mm to (216.5, 125.8)
- moved R33 27.5 mm to (213.0, 125.8)
- moved R34 24.0 mm to (209.5, 125.8)
- moved R35 20.5 mm to (206.0, 125.8)
- moved R36 17.0 mm to (202.5, 125.8)
- moved D20 3.99 mm to (202.5, 129.2), turned to 180 degrees
- moved R13 3.96 mm to (227.0, 130.8)
- moved D19 3.63 mm to (206.0, 129.2), turned to 180 degrees
- moved R20 3.47 mm to (202.5, 130.8)
- moved D18 3.25 mm to (209.5, 129.2), turned to 180 degrees
- moved R14 3.10 mm to (223.5, 130.8)
- moved D24 3.07 mm to (227.0, 127.2), turned to 0 degrees
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- renumbered P2 to J3, P4 to J4, P1 to J5, TP1 to TP10
Connections:
- net Net-(U3-Pad2) renamed /ANALOG_IN
- net Net-(U3-Pad3) renamed /CH_PD
- U3 pad 1: Net-(U3-Pad1) -> /~RESET
- U3 pad 10: Net-(U3-Pad10) -> /SWITCH_3
- U3 pad 12: Net-(U3-Pad12) -> /GPIO0
- U3 pad 13: Net-(U3-Pad13) -> /SWITCH_2
- U3 pad 14: Net-(U3-Pad14) -> /SWITCH_1
- U3 pad 19: Net-(U3-Pad19) -> /SWITCH_5
- U3 pad 20: Net-(U3-Pad20) -> /SWITCH_4
- U3 pad 4: Net-(U3-Pad4) -> /INPUT_1
- U3 pad 5: Net-(U3-Pad5) -> /INPUT_2
- U3 pad 6: Net-(U3-Pad6) -> /INPUT_3
- U3 pad 7: Net-(U3-Pad7) -> /INPUT_4
Routing:
- net /TMP102_PWR: track 40.2 -> 0.00 mm, vias 5 -> 0
- net +5V: track 76.0 -> 39.3 mm, vias 3 -> 2
- net /TMP102_SDA: track 34.2 -> 0.00 mm
- net +3V3: track 28.5 -> 0.00 mm
- net /TMP102_SCL: track 27.8 -> 0.00 mm
- net GND: track 54.0 -> 39.1 mm, vias 26 -> 22
- net /SERIAL_RX: track 9.93 -> 23.0 mm
- net /SERIAL_TX: track 9.93 -> 23.0 mm
- net Net-(J3-Pad8): track 9.96 -> 0.00 mm
- net Net-(J3-Pad6): track 9.93 -> 0.00 mm
- net Net-(J3-Pad4): track 9.89 -> 0.00 mm
- net Net-(J3-Pad2): track 9.86 -> 0.00 mm
- net /~TMP102_ALERT: track 7.38 -> 0.00 mm
- net /INPUT_1: track 23.6 -> 30.7 mm
- net Net-(J3-Pad7): track 4.94 -> 0.00 mm
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Other:
- outline, holes or cut-outs redrawn

Commit message: wip, alpha-2. Routing more or less done.
Parts:
- removed J1: POWER, Pin_Headers:Pin_Header_Straight_2x03_Pitch2.54mm
- removed TP1, TP2, TP3, TP4, TP5, TP6, TP7, TP8: TEST_1P, Connectors_TestPoints:Test_Point_Pad_d1.0mm
- J2: footprint Pin_Headers:Pin_Header_Straight_1x07_Pitch2.54mm -> Pin_Headers:Pin_Header_Straight_1x08_Pitch2.54mm
- moved R37 70.1 mm to (227.2, 115.2), turned to 90 degrees
- moved C8 65.9 mm to (230.6, 126.3), turned to 180 degrees
- moved C7 63.7 mm to (230.7, 116.5), turned to 180 degrees
- moved TP9 62.3 mm to (248.2, 112.8)
- moved U4 56.8 mm to (228.3, 121.2), turned to 180 degrees
- moved J2 48.4 mm to (203.0, 122.0)
- moved R28 5.44 mm to (242.5, 103.5), turned to 0 degrees
- moved R22 3.95 mm to (246.5, 106.5)
- moved R5 3.43 mm to (245.3, 118.8), turned to 180 degrees
- moved R3 3.41 mm to (240.2, 118.8), turned to 180 degrees
- moved R1 3.39 mm to (235.1, 118.8), turned to 180 degrees
- moved R9 3.38 mm to (255.4, 118.8), turned to 180 degrees
- moved R7 3.36 mm to (250.3, 118.8), turned to 180 degrees
- moved R27 3.05 mm to (246.5, 103.5), turned to 0 degrees
- moved R21 2.80 mm to (243.5, 105.5)
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Connections:
- net /CH_PD renamed Net-(U3-Pad3)
- net /TMP102_PWR renamed Net-(P3-Pad7)
- net /TMP102_SCL renamed Net-(P3-Pad5)
- net /TMP102_SDA renamed Net-(P3-Pad3)
- C8 pad 1: +3V3 -> +3.3VP
- J2 pad 2: +3V3 -> +3.3VP
- J2 pad 4: /SERIAL_TX -> /~RESET
- J2 pad 5: /SERIAL_RX -> /ANALOG_IN
- J2 pad 6: /~RESET -> /SERIAL_TX
- J2 pad 7: /GPIO0 -> /SERIAL_RX
- R37 pad 1: +3V3 -> +3.3VP
- U3 pad 10: /SWITCH_3 -> /SWITCH_5
- U3 pad 13: /SWITCH_2 -> /SWITCH_4
- U3 pad 14: /SWITCH_1 -> /SWITCH_3
- U3 pad 19: /SWITCH_5 -> /SWITCH_1
- U3 pad 20: /SWITCH_4 -> /SWITCH_2
- U3 pad 4: /INPUT_1 -> /INPUT_4
- U3 pad 5: /INPUT_2 -> /INPUT_3
- U3 pad 6: /INPUT_3 -> /INPUT_2
- U3 pad 7: /INPUT_4 -> /INPUT_1
- U3 pad 8: +3V3 -> +3.3VP
- U4 pad 2: +3V3 -> +3.3VP
- U4 pad 4: +3V3 -> +3.3VP
Routing:
- net GND: track 39.1 -> 113.8 mm, vias 22 -> 39
- net +5V: track 39.3 -> 110.1 mm, vias 2 -> 4
- net /SWITCH_5: track 31.8 -> 78.9 mm, vias 1 -> 3
- net +3.3VP: track 0.00 -> 46.5 mm
- net /SWITCH_4: track 33.7 -> 74.1 mm, vias 1 -> 3
- net /SWITCH_3: track 40.0 -> 75.8 mm, vias 1 -> 3
- net /INPUT_2: track 20.6 -> 53.6 mm, vias 0 -> 1
- net /INPUT_4: track 19.7 -> 50.5 mm, vias 0 -> 1
- net /INPUT_3: track 22.3 -> 52.9 mm, vias 0 -> 1
- net /INPUT_1: track 30.7 -> 59.4 mm, vias 0 -> 1
- net +3V3: track 0.00 -> 27.8 mm
- net /INPUT_8: track 20.1 -> 46.0 mm, vias 0 -> 1
- net /INPUT_7: track 23.1 -> 46.3 mm, vias 0 -> 1
- net /INPUT_6: track 19.6 -> 42.3 mm, vias 0 -> 1
- net /GPIO0: track 0.00 -> 22.6 mm, vias 0 -> 1
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Other:
- board text added: "Unlock Oslo"
- board text removed: "3.3V"
- board text removed: "5V"
- board text removed: "RX"
- board text removed: "TX"
- board text removed: "Unlock Oslo kommune!"
