File: hardware/alpha-2/alpha.sch (KiCad schematic (older format))
At the start: 107 parts, among them J1 POWER, J10 TEST_1P, J2 SERIAL, J3 TEST_1P, J4 TEST_1P, J5 TEST_1P, J6 TEST_1P, J7 TEST_1P, J8 TEST_1P, J9 TEST_1P, P1 OUTPUTS, P2 INPUTS, P3 RASPBERRY_PI, P4 12V, Q1 DMN2041L-7, Q2 DMN2041L-7, Q3 DMN2041L-7, Q4 DMN2041L-7, Q5 DMN2041L-7, Q6 DMN2041L-7, Q7 DMN2041L-7, U1 TPS54202, U2 TMP102, U3 ESP-12E

Commit message: wip, alpha-2.
Parts:
- removed P1: OUTPUTS, Connectors_Phoenix:PTSA_0,5_12-2,5-Z, symbol Conn_01x12
- removed P2: INPUTS, Connectors_Phoenix:PTSA_0,5_8-2,5-Z, symbol Conn_01x08
- removed P4: 12V, Connectors_Phoenix:PTSA_0,5_2-2,5-Z, symbol Conn_01x02
- removed R24, R25, R26: 10k, IPC7351-Nominal:RESC1005X38, symbol R
- removed U2: TMP102, Bitraf:SOT-563, symbol TMP102
- added J3: INPUTS, Connectors_Phoenix:PTSA_0,5_8-2,5-Z, symbol Conn_01x08
- added J4: 12V, Connectors_Phoenix:PTSA_0,5_2-2,5-Z, symbol Conn_01x02
- added J5: OUTPUTS, Connectors_Phoenix:PTSA_0,5_12-2,5-Z, symbol Conn_01x12
- added R37: 10k, IPC-7351-RESC:RESC_1005x040, symbol R
- C1, C2, C3, C5, C6: footprint IPC7351-Nominal:CAPC2012X70 -> IPC-7351-CAPC:CAPC_2012x125
- C4: footprint IPC7351-Nominal:CAPC1005X55 -> IPC-7351-CAPC:CAPC_1005x050
- C7, C8: renamed from C?; footprint (none) -> IPC-7351-CAPC:CAPC_2012x125
- D10, D12, D2, D24, D25, D26, D27, D28, D29, D30, D31, D4, D6, D8: footprint IPC7351-Nominal:LEDC3216X110 -> IPC-7351-LEDSC:LEDSC_1608x065; ds_Vf 2.0 V -> (none); mpn CMD15-21VRD/TR8 -> SML-D12U1WT86; req_I 5 mA -> 20 mA; req_Vf 1.9V -> 2.2V
- D21, D22, D23: footprint IPC7351-Nominal:LEDC3216X110 -> IPC-7351-LEDSC:LEDSC_1608x065; ds_Vf 2.1 V -> (none); mpn CMD15-21VGD/TR8 -> SML-D12FWT86; req_I 5 mA -> 20 mA; req_Vf 2.0 V -> 2.2 V
- J2: footprint Pin_Headers:Pin_Header_Straight_1x05_Pitch2.54mm -> Pin_Headers:Pin_Header_Straight_1x07_Pitch2.54mm; symbol Conn_01x05 -> Conn_01x07
- R1, R10, R11, R12, R13, R14, R15, R16, R17, R18, R19, R2, R20, R21, R22, R23, R27, R28, R29, R3, R30, R31, R32, R33, R34, R35, R36, R4, R5, R6, R7, R8, R9: footprint IPC7351-Nominal:RESC1005X38 -> IPC-7351-RESC:RESC_1005x040
- TP1: renamed from J3; footprint (none) -> Connectors_TestPoints:Test_Point_Pad_d1.0mm
- TP2: renamed from J4; footprint (none) -> Connectors_TestPoints:Test_Point_Pad_d1.0mm
- TP3: renamed from J5; footprint (none) -> Connectors_TestPoints:Test_Point_Pad_d1.0mm
- TP4: renamed from J6; footprint (none) -> Connectors_TestPoints:Test_Point_Pad_d1.0mm
- TP5: renamed from J7; footprint (none) -> Connectors_TestPoints:Test_Point_Pad_d1.0mm
- TP6: renamed from J8; footprint (none) -> Connectors_TestPoints:Test_Point_Pad_d1.0mm
- TP7: renamed from J9; footprint (none) -> Connectors_TestPoints:Test_Point_Pad_d1.0mm
- TP8: renamed from J10; footprint (none) -> Connectors_TestPoints:Test_Point_Pad_d1.0mm
- TP9: renamed from J?; footprint (none) -> Connectors_TestPoints:Test_Point_Pad_d1.0mm
- U4: renamed from U?; footprint (none) -> smd-semi:SOT-223
- renumbered TP1 to TP10
Connections:
- net +3V3: now also R37.1
- net GND: now also J4.2 (Pin_2)
- net INPUT_1: now also U3.4 (GPIO16)
- net INPUT_2: now also U3.5 (GPIO14)
- net INPUT_3: now also U3.6 (GPIO12)
- net INPUT_4: now also U3.7 (GPIO13)
- net SWITCH_1: now also U3.14 (GPIO5)
- net SWITCH_1_OUT: now also J5.2 (Pin_2)
- net SWITCH_2: now also U3.13 (GPIO4)
- net SWITCH_2_OUT: now also J5.4 (Pin_4)
- net SWITCH_3: now also U3.10 (GPIO15)
- net SWITCH_3_OUT: now also J5.6 (Pin_6)
- net SWITCH_4: now also U3.20 (GPIO10)
- net SWITCH_4_OUT: now also J5.8 (Pin_8)
- net SWITCH_5: now also U3.19 (GPIO9)
- net SWITCH_5_OUT: now also J5.10 (Pin_10)
- net SWITCH_6_OUT: now also J5.12 (Pin_12)
- net Vin: now also J5.1 (Pin_1), J5.11 (Pin_11), J5.3 (Pin_3), J5.5 (Pin_5), J5.7 (Pin_7), J5.9 (Pin_9)
- net at R13.2, TP1.1: now also J3.8 (Pin_8)
- net at R20.2, TP8.1: now also J3.1 (Pin_1)
- net at R19.2, TP7.1: now also J3.2 (Pin_2)
- net at R18.2, TP6.1: now also J3.3 (Pin_3)
- net at R17.2, TP5.1: now also J3.4 (Pin_4)
- net at R16.2, TP4.1: now also J3.5 (Pin_5)
- net at R15.2, TP3.1: now also J3.6 (Pin_6)
- net at R14.2, TP2.1: now also J3.7 (Pin_7)
- net at Q7.3 (D), TP9.1: now also J4.1 (Pin_1)
- net ~RESET: now reaches U3.1 (REST)
- net ~RESET: now also J2.6 (Pin_6)
- net at U3.11 (GPIO2): now also R37.2
- net GPIO0: now reaches U3.12 (GPIO0)
- net GPIO0: now also J2.7 (Pin_7)
- net ANALOG_IN: now reaches U3.2 (ADC)
- net CH_PD: now reaches U3.3 (CH_PD)
- no-connect marks 4 -> 8
Other:
- note added: "ESP8266 BOOT MODES\n GPIO0 GPIO2 GPIO15 \nUART LOW HIGH LOW\nFLASH HIGH HIGH LOW"
- note removed: "Optionally powered by a GPIO pin to reduce self-heating.\n"
- note removed: "Temperature"

Commit message: wip, alpha-2. Routing more or less done.
Parts:
- removed J1: POWER, Pin_Headers:Pin_Header_Straight_2x03_Pitch2.54mm, symbol Conn_02x03_Odd_Even
- removed TP1, TP2, TP3, TP4, TP5, TP6, TP7, TP8: TEST_1P, Connectors_TestPoints:Test_Point_Pad_d1.0mm, symbol TEST_1P
Connections:
- net +3V3: no longer C8.1, J2.2 (Pin_2), R37.1, U3.8 (VCC), U4.2 (Vout), U4.4 (Vout)
- net INPUT_1: now also U3.7 (GPIO13); no longer U3.4 (GPIO16)
- net INPUT_2: now also U3.6 (GPIO12); no longer U3.5 (GPIO14)
- net INPUT_3: now also U3.5 (GPIO14); no longer U3.6 (GPIO12)
- net INPUT_4: now also U3.4 (GPIO16); no longer U3.7 (GPIO13)
- net SWITCH_1: now also U3.19 (GPIO9); no longer U3.14 (GPIO5)
- net SWITCH_2: now also U3.20 (GPIO10); no longer U3.13 (GPIO4)
- net SWITCH_3: now also U3.14 (GPIO5); no longer U3.10 (GPIO15)
- net SWITCH_4: now also U3.13 (GPIO4); no longer U3.20 (GPIO10)
- net SWITCH_5: now also U3.10 (GPIO15); no longer U3.19 (GPIO9)
- new net +3.3VP: C8.1, J2.2 (Pin_2), R37.1, U3.8 (VCC), U4.2 (Vout), U4.4 (Vout)
Other:
- note removed: "Power"

Commit message: o Allowing /.well-known in nginx. o Adding certbot handler for deploying certificates. o Adjusting mosquitto paths for certificates. o Adding handlers for reloading mosquitto config.
Parts:
- J2: footprint Pin_Headers:Pin_Header_Straight_1x07_Pitch2.54mm -> Pin_Headers:Pin_Header_Straight_1x08_Pitch2.54mm; symbol Conn_01x07 -> Conn_01x08
Connections:
- net ANALOG_IN: now also J2.5 (Pin_5)
- net GPIO0: now also J2.8 (Pin_8); no longer J2.7 (Pin_7)
- net SERIAL_RX: now also J2.7 (Pin_7); no longer J2.5 (Pin_5)
- net SERIAL_TX: now also J2.6 (Pin_6); no longer J2.4 (Pin_4)
- net ~RESET: now also J2.4 (Pin_4); no longer J2.6 (Pin_6)
- net CH_PD: no longer names the net of U3.3 (CH_PD)
- net TMP102_PWR: no longer names the net of P3.7 (GPIO4/GCLK)
- net TMP102_SCL: no longer names the net of P3.5 (GPIO3/SCL1)
- net TMP102_SDA: no longer names the net of P3.3 (GPIO2/SDA1)
- no-connect marks 8 -> 17
Changed lines of the file:
@@
 INPUT_1
 $Comp
-L Conn_01x07 J2
+L Conn_01x08 J2
 U 1 1 5A05A056
-P 12600 9300
-F 0 "J2" H 12600 9700 50  0000 C CNN
-F 1 "SERIAL" H 12600 8900 50  0000 C CNN
-F 2 "Pin_Headers:Pin_Header_Straight_1x07_Pitch2.54mm" H 12600 9300 50  0001 C CNN
-F 3 "" H 12600 9300 50  0001 C CNN
-F 4 "footprint only" H 12600 9300 60  0001 C CNN "assembly"
-	1    12600 9300
+P 13000 9200
+F 0 "J2" H 13000 9600 50  0000 C CNN
+F 1 "SERIAL" H 13000 8700 50  0000 C CNN
+F 2 "Pin_Headers:Pin_Header_Straight_1x08_Pitch2.54mm" H 13000 9200 50  0001 C CNN
+F 3 "" H 13000 9200 50  0001 C CNN
+F 4 "footprint only" H 13000 9200 60  0001 C CNN "assembly"
+	1    13000 9200
 	-1   0    0    -1
 $EndComp
@@
 L +5V #PWR05
 U 1 1 5A05A170
-P 12900 8900
-F 0 "#PWR05" H 12900 8750 50  0001 C CNN
-F 1 "+5V" H 12900 9040 50  0000 C CNN
-F 2 "" H 12900 8900 50  0000 C CNN
-F 3 "" H 12900 8900 50  0000 C CNN
-	1    12900 8900
+P 13300 8800
+F 0 "#PWR05" H 13300 8650 50  0001 C CNN
+F 1 "+5V" H 13300 8940 50  0000 C CNN
+F 2 "" H 13300 8800 50  0000 C CNN
+F 3 "" H 13300 8800 50  0000 C CNN
+	1    13300 8800
 	1    0    0    -1
 $EndComp
@@
 L GND #PWR06
 U 1 1 5A05A45F
-P 12900 9700
-F 0 "#PWR06" H 12900 9450 50  0001 C CNN
-F 1 "GND" H 12900 9550 50  0000 C CNN
-F 2 "" H 12900 9700 50  0001 C CNN
-F 3 "" H 12900 9700 50  0001 C CNN
-	1    12900 9700
+P 13300 9700
+F 0 "#PWR06" H 13300 9450 50  0001 C CNN
+F 1 "GND" H 13300 9550 50  0000 C CNN
+F 2 "" H 13300 9700 50  0001 C CNN
+F 3 "" H 13300 9700 50  0001 C CNN
+	1    13300 9700
 	1    0    0    -1
 $EndComp
@@
 	1    0    0    -1
 $EndComp
-Text Label 5100 1500 0    60   ~ 0
-TMP102_SCL
-Text Label 5100 1400 0    60   ~ 0
-TMP102_SDA
 Text Label 5100 2900 0    60   ~ 0
 STATUS_LED_2
@@
 Text Label 8900 1600 2    60   ~ 0
 SERIAL_TX
-Text Label 13600 9300 2    60   ~ 0
+Text Label 14000 9400 2    60   ~ 0
 SERIAL_TX
-Text Label 13600 9400 2    60   ~ 0
+Text Label 14000 9500 2    60   ~ 0
 SERIAL_RX
 NoConn ~ 8100 2600
@@
 Text Label 5100 1800 0    60   ~ 0
 INPUT_8
-Text Label 5100 1600 0    60   ~ 0
-TMP102_PWR
 Text Label 7300 9400 0    60   ~ 0
 SW
@@
 	1    0    0    -1
 $EndComp
-Text Label 5000 4600 0    50   ~ 0
-CH_PD
 Text Label 5000 4400 0    50   ~ 0
 ~RESET
-Text Label 13600 9500 2    50   ~ 0
+Text Label 14000 9200 2    50   ~ 0
 ~RESET
 Text Label 5000 4500 0    50   ~ 0
@@
 	2700 1900 2700 1600
 Wire Wire Line
-	12800 9000 12900 9000
-Wire Wire Line
-	12900 9000 12900 8900
-Wire Wire Line
-	12800 9100 13100 9100
-Wire Wire Line
-	13100 9100 13100 8900
-Wire Wire Line
-	12900 9700 12900 9200
-Wire Wire Line
-	12900 9200 12800 9200
-Wire Wire Line
-	12800 9400 13600 9400
+	13200 8900 13300 8900
+Wire Wire Line
+	13300 8900 13300 8800
+Wire Wire Line
+	13200 9000 13500 9000
+Wire Wire Line
+	13500 9000 13500 8800
+Wire Wire Line
+	13200 9500 14000 9500
 Wire Wire Line
 	9700 10400 9700 10300
@@
 Connection ~ 5700 1300
 Wire Wire Line
-	5900 1400 5100 1400
-Wire Wire Line
-	5900 1500 5100 1500
-Wire Wire Line
 	5900 2900 5100 2900
 Wire Wire Line
@@
 	8900 1700 8100 1700
 Wire Wire Line
-	12800 9300 13600 9300
+	13200 9400 14000 9400
 Wire Wire Line
 	4500 9300 4500 9800
@@
 Wire Wire Line
 	8100 2300 8900 2300
-Wire Wire Line
-	5900 1600 5100 1600
 Wire Wire Line
 	5900 1800 5100 1800
@@
 	7600 5000 8400 5000
 Wire Wire Line
-	12800 9500 13600 9500
+	13200 9200 14000 9200
 Wire Wire Line
 	7600 4600 8400 4600
@@
 	8400 4700 7600 4700
 Wire Wire Line
-	5800 4600 5000 4600
-Wire Wire Line
 	5800 4400 5000 4400
 Wire Wire Line
-	13600 9600 12800 9600
+	14000 9600 13200 9600
 Wire Wire Line
 	5800 4500 5000 4500
@@
 Text Label 8400 4800 2    50   ~ 0
 GPIO0
-Text Label 13600 9600 2    50   ~ 0
+Text Label 14000 9600 2    50   ~ 0
 GPIO0
 $Comp
@@
 L +3.3VP #PWR057
 U 1 1 5A7C3C54
-P 13100 8900
-F 0 "#PWR057" H 13250 8850 50  0001 C CNN
-F 1 "+3.3VP" H 13100 9000 50  0000 C CNN
-F 2 "" H 13100 8900 50  0001 C CNN
-F 3 "" H 13100 8900 50  0001 C CNN
-	1    13100 8900
+P 13500 8800
+F 0 "#PWR057" H 13650 8750 50  0001 C CNN
+F 1 "+3.3VP" H 13500 8900 50  0000 C CNN
+F 2 "" H 13500 8800 50  0001 C CNN
+F 3 "" H 13500 8800 50  0001 C CNN
+	1    13500 8800
 	1    0    0    -1
 $EndComp
@@
 Wire Wire Line
 	7600 7000 7500 7000
+NoConn ~ 8100 2500
+NoConn ~ 8100 2400
+NoConn ~ 5900 2300
+NoConn ~ 5900 2400
+NoConn ~ 5900 2700
+NoConn ~ 5900 1400
+NoConn ~ 5900 1500
+NoConn ~ 5900 1600
+NoConn ~ 5800 4600
+Wire Wire Line
+	13200 9300 14000 9300
+Text Label 14000 9300 2    50   ~ 0
+ANALOG_IN
+Wire Wire Line
+	13200 9100 13300 9100
+Wire Wire Line
+	13300 9100 13300 9700
 $EndSCHEMATC
